File: CerebroPlacaFiltros/CerebroPlaca.sch (KiCad schematic (older format))
At the start: 52 parts

Commit message: se queda con el USB-C
Parts:
- removed J?: USB_OTG-nrfmicro-rescue, symbol cerebro-rescue:USB_OTG-nrfmicro-rescue
Connections:
- wire segments 174 -> 170
- no-connect marks 15 -> 13
Changed lines of the file:
@@
 P0.26
-$Comp
-L cerebro-rescue:USB_OTG-nrfmicro-rescue J?
-U 1 1 5E504B1F
-P 6400 1250
-F 0 "J?" H 6457 1717 50  0000 C CNN
-F 1 "USB_OTG-nrfmicro-rescue" H 6457 1626 50  0000 C CNN
-F 2 "" H 6550 1200 50  0001 C CNN
-F 3 "" H 6550 1200 50  0001 C CNN
-	1    6400 1250
-	1    0    0    -1
-$EndComp
 $Comp
 L Connector:USB_C_Receptacle_USB2.0 J?
@@
 	8900 1150 8800 1150
 Connection ~ 8900 1100
-NoConn ~ 6300 1650
-NoConn ~ 6700 1450
-$Comp
-L nrfmicro-rescue:GND #PWR0115
-U 1 1 5E52C5DE
-P 6500 1650
-F 0 "#PWR0115" H 6500 1400 50  0001 C CNN
-F 1 "GND" V 6505 1522 50  0000 R CNN
-F 2 "" H 6500 1650 50  0001 C CNN
-F 3 "" H 6500 1650 50  0001 C CNN
-	1    6500 1650
-	0    -1   -1   0
-$EndComp
-Wire Wire Line
-	6500 1650 6400 1650
-Text GLabel 6800 1350 2    50   Input ~ 0
-DATA-
-Text GLabel 6800 1250 2    50   Input ~ 0
-DATA+
-Wire Wire Line
-	6700 1250 6800 1250
-Wire Wire Line
-	6800 1350 6700 1350
-Text GLabel 6800 1050 2    50   Input ~ 0
-VBUS
-Wire Wire Line
-	6800 1050 6700 1050
 $Comp
 L cerebro-cache:Connector_Generic_Conn_01x02 J?

Commit message: Reconfig schematic
Parts:
- removed C? (x2): 1uF, symbol Device:C
- removed J?: Connector_Generic_Conn_01x02, symbol cerebro-cache:Connector_Generic_Conn_01x02
- removed JP? (x16): SolderJumper_2_Open, nrfmicro:jumper, symbol Jumper:SolderJumper_2_Open
- added J?: SWD, symbol Connector:Conn_01x04_Male
- added L?: 10uH, symbol Device:L_Small
- added SW?: RESET, symbol Switch:SW_Push
- Q?: symbol AO3407A:AO3407A -> CerebroPlaca-rescue:AO3407A-AO3407A
- SW?: value Switch_SW_SPDT -> Switch; symbol cerebro-cache:Switch_SW_SPDT -> CerebroPlaca-rescue:Switch_SW_SPDT-cerebro-cache
- U?: symbol nrfmicro:E73-2G4M08S1C-52840 -> CerebroPlaca-rescue:E73-2G4M08S1C-52840-nrfmicro
- U?: symbol TI_gv:ADS1294 -> CerebroPlaca-rescue:ADS1294-TI_gv
- Y?: value Crystal -> 32Khz
Connections:
- net labels added: +3V3, +BATT, CLK, CLKSEL, CS, D+, D-, DRDY, DVDD, LED, MISO, MOSI, PWDN, RST, RSTB, RX, SCK, START, SWCLK, SWDCLK, SWDIO, TX
- net labels removed: AVSS, BLUE_LED, BOOT, DATA+, DATA-, DFU, RESET, RESETB, RXD, S1, S2, S3, S4, S5, S6, S7, S8, SPI_CLK, SPI_CS, SPI_DRDY, SPI_IN, SPI_OUT, SPI_START, SW0, SWC, SWD, TXD, VBAT, VCC
- wire segments 170 -> 192
- no-connect marks 13 -> 11
Other:
- note added: "ADS1294"
- note added: "BATTERY CHARGER"
- note added: "MICRONTROLLER"
- note added: "NOTA: Esto es para medir la bateria?\nControl??"
- note added: "NOTA: QUE ES ESTO Y A DONDE VA?"
- note added: "NOTA: REGULADORES PARA AVDD Y DVDD"
- note added: "REGULATOR AND FILTERS"
- note added: "USB & MISSELANOUS"
- moved on the sheet: C?, D?, J?, R?, U?, Y?

Commit message: Fix GND and PWR Reset Resistor
Parts:
- added R? (x2): 10K, symbol Device:R_Small
Connections:
- net labels removed: GNDA
- wire segments 192 -> 201
Changed lines of the file:
@@
 Wire Wire Line
 	1530 5570 2680 5570
-$Comp
-L power:GNDA #PWR?
-U 1 1 5E6A9C8B
-P 4480 4720
-F 0 "#PWR?" H 4480 4470 50  0001 C CNN
-F 1 "GNDA" H 4485 4547 50  0000 C CNN
-F 2 "" H 4480 4720 50  0001 C CNN
-F 3 "" H 4480 4720 50  0001 C CNN
-	1    4480 4720
-	1    0    0    -1
-$EndComp
 Wire Wire Line
 	4380 4420 4480 4420
@@
 Text Label 4470 1720 0    50   ~ 0
 MOSI
-Wire Wire Line
-	4380 2370 4460 2370
-Text Label 4460 2370 0    50   ~ 0
+Text Label 4620 2370 0    50   ~ 0
 RSTB
 Wire Wire Line
@@
 Text Label 4380 2920 0    50   ~ 0
 CLK
-Text Label 4380 2470 0    50   ~ 0
+Text Label 4620 2470 0    50   ~ 0
 PWDN
 Wire Wire Line
@@
 Text Label 1580 5820 0    50   ~ 0
 VREFP
+$Comp
+L Device:R_Small R?
+U 1 1 5E5DCB4C
+P 4420 2220
+F 0 "R?" H 4300 2280 50  0000 L CNN
+F 1 "10K" H 4250 2220 50  0000 L CNN
+F 2 "" H 4420 2220 50  0001 C CNN
+F 3 "~" H 4420 2220 50  0001 C CNN
+	1    4420 2220
+	1    0    0    -1
+$EndComp
+Wire Wire Line
+	4380 2470 4540 2470
+$Comp
+L Device:R_Small R?
+U 1 1 5E5EA517
+P 4540 2220
+F 0 "R?" H 4599 2266 50  0000 L CNN
+F 1 "10K" H 4600 2190 50  0000 L CNN
+F 2 "" H 4540 2220 50  0001 C CNN
+F 3 "~" H 4540 2220 50  0001 C CNN
+	1    4540 2220
+	1    0    0    -1
+$EndComp
+Wire Wire Line
+	4380 2370 4420 2370
+Wire Wire Line
+	4420 2320 4420 2370
+Connection ~ 4420 2370
+Wire Wire Line
+	4420 2370 4620 2370
+Wire Wire Line
+	4540 2320 4540 2470
+Connection ~ 4540 2470
+Wire Wire Line
+	4540 2470 4620 2470
+Wire Wire Line
+	4420 2120 4420 2070
+Wire Wire Line
+	4420 2070 4540 2070
+Wire Wire Line
+	4540 2120 4540 2070
+Connection ~ 4540 2070
+Wire Wire Line
+	4540 2070 4730 2070
+Text Label 4730 2070 0    50   ~ 0
+DVDD
+$Comp
+L power:GND #PWR?
+U 1 1 5E62F77C
+P 4480 4720
+F 0 "#PWR?" H 4480 4470 50  0001 C CNN
+F 1 "GND" H 4485 4547 50  0000 C CNN
+F 2 "" H 4480 4720 50  0001 C CNN
+F 3 "" H 4480 4720 50  0001 C CNN
+	1    4480 4720
+	1    0    0    -1
+$EndComp
 $EndSCHEMATC

Commit message: iniciando
Parts:
- Q?: symbol CerebroPlaca-rescue:AO3407A-AO3407A -> CerebroPlaca-rescue:AO3407A-AO3407A-CerebroPlaca-rescue
- SW?: symbol CerebroPlaca-rescue:Switch_SW_SPDT-cerebro-cache -> CerebroPlaca-rescue:Switch_SW_SPDT-cerebro-cache-CerebroPlaca-rescue
- U?: symbol CerebroPlaca-rescue:E73-2G4M08S1C-52840-nrfmicro -> CerebroPlaca-rescue:E73-2G4M08S1C-52840-nrfmicro-CerebroPlaca-rescue
- U?: symbol CerebroPlaca-rescue:ADS1294-TI_gv -> CerebroPlaca-rescue:ADS1294-TI_gv-CerebroPlaca-rescue
Changed lines of the file:
@@
 EESchema Schematic File Version 4
+LIBS:CerebroPlaca-cache
 EELAYER 30 0
 EELAYER END
@@
 $EndDescr
 $Comp
-L CerebroPlaca-rescue:E73-2G4M08S1C-52840-nrfmicro U?
+L CerebroPlaca-rescue:E73-2G4M08S1C-52840-nrfmicro-CerebroPlaca-rescue U?
 U 1 1 5E4D9260
 P 9690 2220
@@
 	8690 1220 8990 1220
 $Comp
-L CerebroPlaca-rescue:GND-nrfmicro-rescue #PWR0101
+L CerebroPlaca-rescue:GND-nrfmicro-rescue-CerebroPlaca-rescue #PWR0101
 U 1 1 5E4DE4C5
 P 8690 1520
@@
 	8340 3220 8990 3220
 $Comp
-L CerebroPlaca-rescue:GND-nrfmicro-rescue #PWR0104
+L CerebroPlaca-rescue:GND-nrfmicro-rescue-CerebroPlaca-rescue #PWR0104
 U 1 1 5E4E325C
 P 10490 3120
@@
 $EndComp
 $Comp
-L CerebroPlaca-rescue:GND-nrfmicro-rescue #PWR0105
+L CerebroPlaca-rescue:GND-nrfmicro-rescue-CerebroPlaca-rescue #PWR0105
 U 1 1 5E4E79AC
 P 6520 3410
@@
 	6680 7390 6580 7390
 $Comp
-L CerebroPlaca-rescue:GND-nrfmicro-rescue #PWR0106
+L CerebroPlaca-rescue:GND-nrfmicro-rescue-CerebroPlaca-rescue #PWR0106
 U 1 1 5E4EF534
 P 5730 7490
@@
 $EndComp
 $Comp
-L CerebroPlaca-rescue:GND-nrfmicro-rescue #PWR0107
+L CerebroPlaca-rescue:GND-nrfmicro-rescue-CerebroPlaca-rescue #PWR0107
 U 1 1 5E4F4E0F
 P 6780 6890
@@
 $EndComp
 $Comp
-L CerebroPlaca-rescue:GND-nrfmicro-rescue #PWR0109
+L CerebroPlaca-rescue:GND-nrfmicro-rescue-CerebroPlaca-rescue #PWR0109
 U 1 1 5E4FC8BD
 P 7350 5560
@@
 	7350 5460 7350 5560
 $Comp
-L CerebroPlaca-rescue:GND-nrfmicro-rescue #PWR0110
+L CerebroPlaca-rescue:GND-nrfmicro-rescue-CerebroPlaca-rescue #PWR0110
 U 1 1 5E4FE7F8
 P 6800 5560
@@
 	6250 5110 6250 5160
 $Comp
-L CerebroPlaca-rescue:GND-nrfmicro-rescue #PWR0111
+L CerebroPlaca-rescue:GND-nrfmicro-rescue-CerebroPlaca-rescue #PWR0111
 U 1 1 5E50568F
 P 5850 5660
@@
 $EndComp
 $Comp
-L CerebroPlaca-rescue:GND-nrfmicro-rescue #PWR0112
+L CerebroPlaca-rescue:GND-nrfmicro-rescue-CerebroPlaca-rescue #PWR0112
 U 1 1 5E507D22
 P 5500 5660
@@
 Connection ~ 5500 5110
 $Comp
-L CerebroPlaca-rescue:AO3407A-AO3407A Q?
+L CerebroPlaca-rescue:AO3407A-AO3407A-CerebroPlaca-rescue Q?
 U 1 1 5E4E6AE3
 P 6150 4660
@@
 	5350 5110 5250 5110
 $Comp
-L CerebroPlaca-rescue:Switch_SW_SPDT-cerebro-cache SW?
+L CerebroPlaca-rescue:Switch_SW_SPDT-cerebro-cache-CerebroPlaca-rescue SW?
 U 1 1 5E4F24BD
 P 6600 4510
@@
 NoConn ~ 5540 2680
 $Comp
-L CerebroPlaca-rescue:GND-nrfmicro-rescue #PWR0113
+L CerebroPlaca-rescue:GND-nrfmicro-rescue-CerebroPlaca-rescue #PWR0113
 U 1 1 5E50D022
 P 5940 2680
@@
 $EndComp
 $Comp
-L CerebroPlaca-rescue:GND-nrfmicro-rescue #PWR0114
+L CerebroPlaca-rescue:GND-nrfmicro-rescue-CerebroPlaca-rescue #PWR0114
 U 1 1 5E51E12E
 P 7290 1430
@@
 	4480 4520 4480 4620
 $Comp
-L CerebroPlaca-rescue:GND-nrfmicro-rescue #PWR?
+L CerebroPlaca-rescue:GND-nrfmicro-rescue-CerebroPlaca-rescue #PWR?
 U 1 1 5E50718C
 P 920 2130
@@
 $EndComp
 $Comp
-L CerebroPlaca-rescue:ADS1294-TI_gv U?
+L CerebroPlaca-rescue:ADS1294-TI_gv-CerebroPlaca-rescue U?
 U 1 1 5E4E799B
 P 3430 3720

Commit message: el esquematico esta casi listo, solo falta la footprin del ads1294
Parts:
- added C1, C10, C3, C4: 10uf, Capacitor_SMD:C_0805_2012Metric, symbol Device:C
- added C11, C2: 2.2uF, Capacitor_SMD:C_0805_2012Metric, symbol Device:C
- added C12, C15: 1uF, Capacitor_SMD:C_0805_2012Metric, symbol Device:C
- added C16, C18: 0.1uF, Capacitor_SMD:C_0805_2012Metric, symbol Device:C
- added L1, L2: 3.3uH, Inductor_SMD:L_7.3x7.3_H3.5, symbol Device:L
- added U1, U3: TPS73250DBVT, footprints:TPS73250DBVT, symbol tps73250dbvt:TPS73250DBVT
- C13, C14, C17, C19, C20, C21, C22, C5, C6, C7, C8, C9: renamed from C?; footprint (none) -> Capacitor_SMD:C_0805_2012Metric
- D1: renamed from D?; footprint Diode_THT:D_DO-41_SOD81_P10.16mm_Horizontal -> Diode_SMD:D_SOD-123F
- D2, D3: renamed from D?; footprint (none) -> LED_SMD:LED_0603_1608Metric
- J1: renamed from J?; footprint (none) -> Connector_PinHeader_1.00mm:PinHeader_1x04_P1.00mm_Vertical
- J2: renamed from J?; footprint (none) -> nrfmicro:usb_type_c
- L3: renamed from L?; footprint (none) -> Inductor_SMD:L_7.3x7.3_H3.5
- Q1: renamed from Q?; footprint SOT95P280X125-3N -> Package_TO_SOT_SMD:SOT-23
- R1, R10, R11, R2, R3, R4, R5, R6, R7, R8, R9: renamed from R?; footprint (none) -> Resistor_SMD:R_0603_1608Metric
- SW1: renamed from SW?; footprint (none) -> nrfmicro:switch_MSK-12C02_smd
- SW2: renamed from SW?; footprint (none) -> Button_Switch_SMD:SW_SPST_TL3342
- U6: renamed from U?; footprint (none) -> nrfmicro:E73-2G4M08S1C
- Y1: renamed from Y?; footprint (none) -> Crystal:Crystal_Round_D1.0mm_Vertical
- gave numbers to parts that had none: 3
Connections:
- net AVDD: now also C1.1, C15.1, C18.1, C4.1, L1.2, L2.2
- net DVDD: now also C12.1, C16.1
- net GND: now also C19.1, C1.2, C10.2, C11.2, C12.2, C15.2, C16.2, C18.2, C2.2, C3.2, C4.2, U1.2 (GND), U3.2 (GND); no longer C19.2
- net Electodo_1_-: now reaches U2.15 (IN1N)
- net Electodo_1_+: now reaches U2.16 (IN1P)
- net at U2.64 (WCT): now also C19.2; no longer C19.1
- new net: C10.1, C11.1, L1.1, U3.5 (OUT)
- new net: C2.1, C3.1, L2.1, U1.5 (OUT)
- new net VCC: U1.1 (IN), U1.3 (EN), U3.1 (IN), U3.3 (EN)
- no-connect marks 11 -> 13
Other:
- note removed: "NOTA: QUE ES ESTO Y A DONDE VA?"
- moved on the sheet: C19

Commit message: Tanto esquematico como pcb, preparados
Parts:
- added J3: Conn_01x03_Male, Connector_PinHeader_1.00mm:PinHeader_1x03_P1.00mm_Vertical, symbol Connector:Conn_01x03_Male
- U2: footprint (none) -> ADS1294IPAG:ADS1294IPAG
Connections:
- net Electodo_1_+: now also J3.3 (Pin_3)
- net Electodo_1_-: now also J3.2 (Pin_2)
- net GND: now also J3.1 (Pin_1)
Other:
- note added: "Electrodos"
Changed lines of the file:
@@
 F 0 "U2" H 3530 6357 60  0000 C CNN
 F 1 "ADS1294" H 3530 6251 60  0000 C CNN
-F 2 "" H 3430 3720 60  0000 C CNN
+F 2 "ADS1294IPAG:ADS1294IPAG" H 3920 3530 60  0000 C CNN
 F 3 "" H 3430 3720 60  0000 C CNN
 	1    3430 3720
@@
 	1    0    0    -1
 $EndComp
+Wire Notes Line
+	9500 6540 9500 5340
+Wire Notes Line
+	9500 5340 11220 5340
+Text Notes 10150 5490 0    50   ~ 0
+Electrodos
+$Comp
+L Connector:Conn_01x03_Male J3
+U 1 1 5E6AA605
+P 10510 5930
+F 0 "J3" H 10482 5862 50  0000 R CNN
+F 1 "Conn_01x03_Male" H 10482 5953 50  0000 R CNN
+F 2 "Connector_PinHeader_1.00mm:PinHeader_1x03_P1.00mm_Vertical" H 10510 5930 50  0001 C CNN
+F 3 "~" H 10510 5930 50  0001 C CNN
+	1    10510 5930
+	-1   0    0    1
+$EndComp
+$Comp
+L nrfmicro-rescue:GND #PWR01
+U 1 1 5E6AD0C0
+P 9880 6090
+F 0 "#PWR01" H 9880 5840 50  0001 C CNN
+F 1 "GND" H 9885 5917 50  0000 C CNN
+F 2 "" H 9880 6090 50  0001 C CNN
+F 3 "" H 9880 6090 50  0001 C CNN
+	1    9880 6090
+	1    0    0    -1
+$EndComp
+Wire Wire Line
+	9880 6090 10310 6090
+Wire Wire Line
+	10310 6090 10310 6030
+Text Label 9740 5830 0    50   ~ 0
+Electodo_1_+
+Text Label 9740 5930 0    50   ~ 0
+Electodo_1_-
+Wire Wire Line
+	9740 5930 10310 5930
+Wire Wire Line
+	10310 5830 9740 5830
 $EndSCHEMATC
