File: CerebroPlaca/CerebroPlaca.kicad_pcb (KiCad board)
At the start: 2 copper layers, 309.9 x 255.3 mm, 40 parts, among them J1 Connector_Generic_Conn_01x02, J2 USB_C_Receptacle_USB2.0, J3 Conn_01x08_Male, Q1 AO3407A, SW1 Switch_SW_SPDT, U1 AP2112K-3.3, U2 E73-2G4M08S1C-52840, U3 MCP73831-2-OT, Y1 Crystal

Commit message: ajustes en placaCerebro
Parts:
- removed JP1, JP10, JP11, JP12, JP13, JP14, JP15, JP16, JP2, JP3, JP4, JP5, JP6, JP7, JP8, JP9: SolderJumper_2_Open, nrfmicro:jumper
- added L1: 10uH, Inductor_SMD:L_7.3x7.3_H3.5, F.Cu at (130.2, 102.8)
- added SW2: RESET, Button_Switch_SMD:SW_SPST_TL3342, F.Cu at (138.0, 102.1)
- J1: value Connector_Generic_Conn_01x02 -> Conn_01x04_Male; footprint nrfmicro:connector_swd -> Connector_PinHeader_1.00mm:PinHeader_1x04_P1.00mm_Vertical
- Y1: value Crystal -> 32Khz
- moved Ref** 71.7 mm to (127.0, 150.5)
- moved J1 58.7 mm to (128.5, 109.3)
- moved R1 56.2 mm to (124.8, 115.0)
- moved C3 51.4 mm to (121.4, 116.1)
- moved R8 44.2 mm to (132.1, 112.0)
- moved C2 41.1 mm to (124.5, 109.3), turned to 180 degrees
- moved U1 38.0 mm to (123.1, 104.5)
- moved R4 36.1 mm to (119.5, 104.5), turned to 270 degrees
- moved C1 36.0 mm to (120.8, 109.3), turned to 0 degrees
- moved J2 34.3 mm to (151.4, 89.6)
- moved J3 34.1 mm to (124.9, 71.9)
- moved R2 33.8 mm to (119.5, 99.7)
- moved SW1 33.8 mm to (110.3, 96.1), turned to 0 degrees
- moved D1 33.1 mm to (116.3, 106.7), turned to 180 degrees
- moved Q1 32.8 mm to (116.4, 102.2), turned to 90 degrees
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Connections:
- net BLUE_LED renamed /LED
- net DATA+ renamed /D+
- net DATA- renamed /D-
- net DFU renamed Net-(U2-Pad38)
- net Net-(U2-Pad10) renamed /PWDN
- net Net-(U2-Pad28) renamed /MISO
- net Net-(U2-Pad4) renamed /RSTB
- net Net-(U2-Pad7) renamed /CS
- net Net-(U2-Pad8) renamed /START
- net Net-(U2-Pad9) renamed /DRDY
- net P0.03 renamed /P0.03
- net P1.04 renamed /P1.04
- net P1.09 renamed /P1.09
- net P1.11 renamed /P1.11
- net VBAT renamed /+BATT
- C2 pad 1: VCC -> +3V3
- J1 pad 1: SWD -> +3V3
- J1 pad 2: SWC -> /SWDIO
- J3 pad 2: P1.06 -> /P0.13
- J3 pad 5: P1.13 -> /P0.20
- J3 pad 7: VBUS -> +3V3
- U1 pad 5: VCC -> +3V3
- U2 pad 14: TXD -> /TXD
- U2 pad 16: RXD -> /RXD
- U2 pad 19: VCC -> +3V3
- U2 pad 23: Net-(U2-Pad23) -> +3V3
- U2 pad 26: RESET -> /RST
- U2 pad 32: Net-(U2-Pad32) -> /P0.20
- U2 pad 33: Net-(U2-Pad33) -> /P0.13
- U2 pad 37: SWD -> /SWDIO
- U2 pad 39: SWC -> /SWDCLK
- U2 pad 42: P1.06 -> /MOSI
- U2 pad 6: P1.13 -> /SCK
Routing:
- net Net-(R6-Pad1): track 2.05 -> 83.7 mm
- net +3V3: track 0.00 -> 75.6 mm, vias 0 -> 2
- net VCC: track 36.7 -> 0.00 mm, vias 2 -> 0
- net /P0.13: track 0.00 -> 29.5 mm, vias 0 -> 2
- net /SWDIO: track 0.00 -> 28.7 mm, vias 0 -> 2
- net TXD: track 25.8 -> 0.00 mm, vias 2 -> 0
- net GND: track 154.2 -> 128.6 mm, vias 3 -> 2
- net P1.13: track 23.7 -> 0.00 mm, vias 1 -> 0
- net Net-(J2-PadB5): track 22.8 -> 46.1 mm
- net /P0.20: track 0.00 -> 23.0 mm, vias 0 -> 2
- net VBUS: track 100.6 -> 81.9 mm
- net RXD: track 16.3 -> 0.00 mm, vias 2 -> 0
- net P1.06: track 15.4 -> 0.00 mm, vias 1 -> 0
- net Net-(J2-PadA5): track 18.1 -> 3.93 mm
- net Net-(Q1-Pad3): track 18.5 -> 7.56 mm
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
Commit message: ajuste de la placa a 7.5 cm de ancho
Parts:
- removed the Ref** at (127.0, 150.5)
- added Ref**: Val**, CerebroInkscape, F.Cu at (118.1, 93.7)
- moved J2 69.7 mm to (81.8, 87.6), turned to 90 degrees
- moved J3 47.6 mm to (137.4, 117.8), turned to 270 degrees
- moved C3 33.0 mm to (147.3, 95.6), turned to 270 degrees
- moved R1 31.3 mm to (146.2, 92.2), turned to 0 degrees
- moved R6 29.5 mm to (133.0, 74.0), turned to 180 degrees
- moved R8 29.3 mm to (143.2, 84.9), turned to 90 degrees
- moved U3 28.5 mm to (144.1, 95.4), turned to 90 degrees
- moved D3 27.7 mm to (129.3, 74.0), turned to 180 degrees
- moved R5 27.6 mm to (143.2, 88.7), turned to 90 degrees
- moved J1 24.0 mm to (140.5, 88.5), turned to 180 degrees
- moved SW2 23.6 mm to (133.3, 79.0), turned to 180 degrees
- moved C1 23.6 mm to (140.5, 96.2), turned to 90 degrees
- moved C2 23.2 mm to (140.5, 92.5), turned to 270 degrees
- moved R7 22.6 mm to (123.3, 76.9), turned to 180 degrees
- moved D1 22.4 mm to (137.9, 100.7), turned to 270 degrees
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Routing:
- net Net-(J2-PadB5): track 46.1 -> 109.1 mm
- net /P0.13: track 29.5 -> 73.6 mm, vias 2 -> 0
- net GND: track 128.6 -> 168.7 mm, vias 2 -> 4
- net VBUS: track 81.9 -> 117.4 mm
- net Net-(J2-PadA5): track 3.93 -> 36.9 mm
- net /P1.04: track 13.7 -> 40.7 mm, vias 0 -> 2
- net /P0.20: track 23.0 -> 46.3 mm
- net /P1.11: track 17.5 -> 40.5 mm
- net /D+: track 17.2 -> 38.8 mm, vias 0 -> 2
- net /P0.03: track 14.5 -> 35.4 mm, vias 0 -> 2
- net /D-: track 18.7 -> 39.4 mm
- net +3V3: track 75.6 -> 65.5 mm, vias 2 -> 3
- net /P1.09: track 31.3 -> 33.3 mm
- net /SWDIO: track 28.7 -> 30.2 mm
- removed copper zone on B.Cu, net (none)
- removed copper zone on F.Cu, net (none)
Other:
- board size 309.9 x 255.3 mm -> 75 x 61.8 mm

Commit message: ajusted de placa
Routing:
- added copper zone on B.Cu, net (none)
- added copper zone on F.Cu, net (none)
Changed lines of the file:
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@@
   (segment (start 131.9614 83.6377) (end 130.0695 85.5296) (width 0.25) (layer F.Cu) (net 43))
   (segment (start 134.0319 83.6377) (end 131.9614 83.6377) (width 0.25) (layer F.Cu) (net 43))
+  (zone (net 0) (net_name "") (layer F.Cu) (hatch edge 0.508)
+    (connect_pads (clearance 0.508))
+    (min_thickness 0.254)
+    (fill yes (arc_segments 32) (thermal_gap 0.508) (thermal_bridge_width 0.508))
+    (polygon
+      (pts
+        (xy 74 62.4) (xy 154.9 62.3) (xy 156.2 123.3) (xy 96.2 126.4) (xy 73 82.8)
+      )
+    )
+  )
+  (zone (net 0) (net_name "") (layer B.Cu) (hatch edge 0.508)
+    (connect_pads (clearance 0.508))
+    (min_thickness 0.254)
+    (fill yes (arc_segments 32) (thermal_gap 0.508) (thermal_bridge_width 0.508))
+    (polygon
+      (pts
+        (xy 156.5 125.4) (xy 112 127.8) (xy 89.9 106.5) (xy 74.9 85.6) (xy 98.6 54.6)
+        (xy 156.8 65.4)
+      )
+    )
+  )
 )
